Commit message: fix(examples): lift the flag vane clear of its base
The vane's collision box sat inside the base's. MuJoCo does not filter
contacts between a joint's child and a parent welded to the world, so
the contacts took 0.12 of the SG90's 0.128 N·m and the flag crawled at
about 107°/s at near-stall current. Browser QA of the vcc world showed
the rail pinned at 4.32 V.

The hinge sits 0.5 mm above the base now, and the flag cruises at about
496°/s. The limit widens to pi so the vcc sketch's 170° swing stays off
the stop.

Co-Authored-By: Claude Opus 5.5 <noreply@anthropic.com>

File: examples/nano/robot/flag.urdf (robot description, URDF)
Before this commit: robot flag, 2 links, 1 joints
Joints:
- joint hinge: limit lower=0 upper=2.617993877991494 effort=0.18 velocity=10.472 -> lower=0 upper=3.141592653589793 effort=0.18 velocity=10.472; origin xyz=0 0 0.0125 rpy=0 0 0 -> xyz=0 0 0.023 rpy=0 0 0
